File: schematics/byggern.sch (KiCad schematic (older format))
At the start: 5 parts

Commit message: Further work on sch
Parts:
- added C? (x3): C, symbol C
- 4.9MHz1: renamed from 4.9MHz; footprint (none) -> Crystals:crystal_FA238-TSX3225
- IC1: renamed from IC?; footprint DIL40 -> Housings_DIP:DIP-40_W15.24mm
- IC2: renamed from IC?; footprint (none) -> Housings_DIP:DIP-28_W7.62mm
- U1, U2: renamed from U?; footprint (none) -> Housings_DIP:DIP-20_W7.62mm
Connections:
- net labels added: ALE, D0, D1, D2, D3, D4, D5, D6, D7
- wire segments 22 -> 48
Other:
- moved on the sheet: 4.9MHz1, IC1, IC2, U1

Commit message: Added the MAX Chip
Parts:
- added C? (x3): C, symbol C
- added U?: MAX233, symbol MAX233
Connections:
- wire segments 48 -> 50
Changed lines of the file:
@@
 LIBS:valves
 LIBS:byggern
-LIBS:byggern-cache
 EELAYER 25 0
 EELAYER END
@@
 Text Label 5600 1600 2    47   ~ 0
 D7
+$Comp
+L C C?
+U 1 1 57D6B4C0
+P 2000 2850
+F 0 "C?" H 2025 2950 50  0000 L CNN
+F 1 "C" H 2025 2750 50  0000 L CNN
+F 2 "" H 2038 2700 50  0000 C CNN
+F 3 "" H 2000 2850 50  0000 C CNN
+	1    2000 2850
+	0    -1   -1   0
+$EndComp
+$Comp
+L C C?
+U 1 1 57D6B509
+P 2000 3250
+F 0 "C?" H 2025 3350 50  0000 L CNN
+F 1 "C" H 2025 3150 50  0000 L CNN
+F 2 "" H 2038 3100 50  0000 C CNN
+F 3 "" H 2000 3250 50  0000 C CNN
+	1    2000 3250
+	0    -1   -1   0
+$EndComp
+$Comp
+L GND #PWR?
+U 1 1 57D6B646
+P 1750 2850
+F 0 "#PWR?" H 1750 2600 50  0001 C CNN
+F 1 "GND" H 1750 2700 50  0000 C CNN
+F 2 "" H 1750 2850 50  0000 C CNN
+F 3 "" H 1750 2850 50  0000 C CNN
+	1    1750 2850
+	0    1    1    0
+$EndComp
+$Comp
+L GND #PWR?
+U 1 1 57D6B673
+P 1750 3250
+F 0 "#PWR?" H 1750 3000 50  0001 C CNN
+F 1 "GND" H 1750 3100 50  0000 C CNN
+F 2 "" H 1750 3250 50  0000 C CNN
+F 3 "" H 1750 3250 50  0000 C CNN
+	1    1750 3250
+	0    1    1    0
+$EndComp
+$Comp
+L MAX233 U?
+U 1 1 57D6BDDF
+P 1100 6450
+F 0 "U?" H 1900 6550 60  0000 C CNN
+F 1 "MAX233" H 1900 6650 60  0000 C CNN
+F 2 "" H 1650 7350 60  0001 C CNN
+F 3 "" H 1650 7350 60  0001 C CNN
+	1    1100 6450
+	1    0    0    -1
+$EndComp
 Wire Wire Line
 	9600 4350 9600 4500
@@
 	2350 3200 2350 3250
 Wire Wire Line
-	2350 3250 2450 3250
-Wire Wire Line
-	2450 2850 2350 2850
+	2150 3250 2450 3250
+Wire Wire Line
+	2150 2850 2450 2850
 Wire Wire Line
 	2350 2850 2350 2900
@@
 Wire Wire Line
 	9000 4050 8850 4050
+Connection ~ 2350 2850
+Connection ~ 2350 3250
+Wire Wire Line
+	1750 3250 1850 3250
+Wire Wire Line
+	1850 2850 1750 2850
+$Comp
+L C C?
+U 1 1 57D6DE08
+P 1250 7000
+F 0 "C?" H 1275 7100 50  0000 L CNN
+F 1 "C" H 1275 6900 50  0000 L CNN
+F 2 "" H 1288 6850 50  0000 C CNN
+F 3 "" H 1250 7000 50  0000 C CNN
+	1    1250 7000
+	1    0    0    -1
+$EndComp
 $EndSCHEMATC

Commit message: Updated to reflex ex-2
Parts:
- added 4.7k: R, symbol R
- added C? (x2): C, symbol C
- added SW?: SW_PUSH, symbol SW_PUSH
- added U?: RS232-Pinouts, symbol RS232-Pinouts
- added U?: MC78L05AACP, TO-92, symbol MC78L05AACP
- renumbered 4.9MHz1 to 4.9MHz
Connections:
- net +5V: now also C?.2, U?.7 (VCC), 4.7k.2, C?.1, U?.1 (OUT)
- net GND: now also C?.1, U?.6 (GND), U?.9 (GND), C?.2, C?.2, SW?.1, U?.14 (GND), U?.2 (GND), U?.6 (GND)
- net RD: now reaches IC2.22 (~OE~)
- net RD: now also IC1.17 ((~RD~)PD7)
- net at IC2.26 (CS2): now also U2.19 (I/O/Q)
- net WR: now reaches IC2.27 (~WR~)
- net WR: now also IC1.16 ((~WR~)PD6)
- net at U2.1 (I/CLK): now also IC1.24 ((PCINT11/A11)PC3)
- net at U2.2 (I): now also IC1.23 ((PCINT10/A10)PC2)
- net at IC1.10 ((RXD0)PD0): now also U?.3 (R1OUT)
- net at IC1.11 ((TXD0)PD1): now also U?.2 (T1IN)
- net at IC1.9 (~RESET): now also 4.7k.1, SW?.2
- net at U?.10 ((V-)CS-): now also U?.16 (C2-)
- net at U?.11 (C2+(C2-)): now also U?.15 (C2+)
- net at U?.12 (V-(C2+)): now also U?.17 (V-)
- net at U?.4 (R1IN): now also U?.1 (TX)
- net at U?.5 (T1OUT): now also U?.2 (RX)
- new net +12V: C?.1, U?.3 (IN)
Other:
- note added: "Power Supply"
- moved on the sheet: C?, U?
