File: schematics/byggern.sch (KiCad schematic (older format))
At the start: 19 parts, among them IC1 ATMEGA162-P, IC2 CY7C185, U1 74LS573, U2 GAL16V8D

Commit message: Updated the schematics to represent the lab
Parts:
- removed U?: MultiFunctionCard, symbol MultiFunctionCard
- added 16kHz: Crystal, Crystals:crystal_FA238-TSX3225, symbol Crystal
- added C? (x3): C, symbol C
- added U?: MultiFunctionCard, symbol MultiFunctionCard
- added U?: MCP2515, symbol MCP2515
- added U?: ADC0844, symbol ADC0844
Connections:
- net +5V: now also C?.2, U?.13 (VCC), U?.20 (Vcc)
- net D0: now also U?.4 (OLED-D1)
- net D1: now also U?.5 (OLED-D2)
- net D2: now also U?.6 (OLED-D3)
- net D3: now also U?.7 (OLED-D4)
- net D4: now also U?.8 (OLED-D5)
- net D5: now also U?.9 (OLED-D6)
- net D6: now also U?.10 (OLED-D7)
- net D7: now also U?.11 (OLED-D8)
- net GND: now also IC1.28 ((PCINT15/TDI/A15)PC7), C?.1, C?.2, C?.2, U?.10 (DGND), U?.12 (OLED-GND), U?.14 (GND), U?.7 (AGND), U?.8 (V_ref)
- net at U2.1 (I/CLK): now also IC1.27 ((PCINT14/TDO/A14)PC6); no longer IC1.28 ((PCINT15/TDI/A15)PC7)
- net OLED-~CS: now reaches U2.17 (I/O/Q)
- net OLED-~CS: now also U?.1 (OLED-~CS)
- net ADC-~CS: now reaches U2.18 (I/O/Q)
- net ADC-~CS: now also U?.2 (~CS)
- net at U2.2 (I): now also IC1.26 ((PCINT13/TMS/A13)PC5); no longer IC1.27 ((PCINT14/TDO/A14)PC6)
- net AT-RX: now reaches IC1.10 ((RXD0)PD0), U?.3 (R1OUT)
- net AT-TX: now reaches IC1.11 ((TXD0)PD1), U?.2 (T1IN)
- net ~SS: now reaches IC1.5 ((OC3B/~SS~)PB4)
- net ~SS: now also U?.16 (~CS)
- net MOSI: now reaches IC1.6 ((MOSI)PB5)
- net MOSI: now also U?.14 (SI)
- net MISO: now reaches IC1.7 ((MISO)PB6)
- net MISO: now also U?.15 (SO)
- net SCK: now reaches IC1.8 ((SCK)PB7)
- net SCK: now also U?.13 (SCK)
- net RD renamed ~RD
- net ~RD: now also U?.19 (~WR)
- net WR renamed ~WR
- net ~WR: now also U?.1 (~RD), U?.3 (OLED-R/~W)
- new net: 16kHz.1, C?.1, U?.7 (OSC2)
- new net: 16kHz.2, C?.1, U?.8 (OSC1)
- new net ??: U?.2 (OLED-~D~/C)
- new net DB0: U?.17 (DB0/MA0)
- new net DB1: U?.16 (DB1/MA1)
- new net DB2: U?.15 (DB2/MA2)
- new net DB3: U?.14 (DB3/MA3)
- new net DB4: U?.13 (DB4)
- new net DB5: U?.12 (DB5)
- new net DB6: U?.11 (DB6)
- new net DB7: U?.9 ((MSB)DB7)
Other:
- note added: "ADC"
- note added: "CAN Controller"
- note added: "Data/Addr Bus"
- note added: "UART and RS232"
- note added: "USB Multifunction Card"
- moved on the sheet: C?, U?
