File: schematics/_saved_byggern.sch (KiCad schematic (older format))
At the start: 19 parts, among them IC1 ATMEGA162-P, IC2 CY7C185, U1 74LS573, U2 GAL16V8D

Commit message: dd
Connections:
- net at U2.1 (I/CLK): no longer IC1.28 ((PCINT15/TDI/A15)PC7)
- net at U2.2 (I): no longer IC1.27 ((PCINT14/TDO/A14)PC6)
Changed lines of the file:
@@
 	2350 3200 2350 3250
 Wire Wire Line
-	2150 3250 2350 3250
-Wire Wire Line
-	2350 3250 2450 3250
-Wire Wire Line
-	2150 2850 2350 2850
-Wire Wire Line
-	2350 2850 2450 2850
+	2150 3250 2450 3250
+Wire Wire Line
+	2150 2850 2450 2850
 Wire Wire Line
 	2350 2850 2350 2900
@@
 	9000 3050 7750 3050
 Wire Wire Line
-	4450 2350 4550 2350
-Wire Wire Line
-	4550 2350 6350 2350
-Wire Wire Line
-	4450 2450 4700 2450
-Wire Wire Line
-	4700 2450 6350 2450
-Wire Wire Line
-	4450 2550 4850 2550
-Wire Wire Line
-	4850 2550 6350 2550
-Wire Wire Line
-	4450 2650 5000 2650
-Wire Wire Line
-	5000 2650 6350 2650
-Wire Wire Line
-	4450 2750 5150 2750
-Wire Wire Line
-	5150 2750 6350 2750
-Wire Wire Line
-	4450 2850 5300 2850
-Wire Wire Line
-	5300 2850 6350 2850
-Wire Wire Line
-	4450 2950 5450 2950
-Wire Wire Line
-	5450 2950 6350 2950
-Wire Wire Line
-	4450 3050 5600 3050
-Wire Wire Line
-	5600 3050 6350 3050
+	4450 2350 6350 2350
+Wire Wire Line
+	4450 2450 6350 2450
+Wire Wire Line
+	4450 2550 6350 2550
+Wire Wire Line
+	4450 2650 6350 2650
+Wire Wire Line
+	4450 2750 6350 2750
+Wire Wire Line
+	4450 2850 6350 2850
+Wire Wire Line
+	4450 2950 6350 2950
+Wire Wire Line
+	4450 3050 6350 3050
 Wire Bus Line
-	10450 1450 10450 2250
+	10450 1450 10450 2950
 Wire Bus Line
-	10450 2250 10450 2350
-Wire Bus Line
-	10450 2350 10450 2450
-Wire Bus Line
-	10450 2450 10450 2550
-Wire Bus Line
-	10450 2550 10450 2650
-Wire Bus Line
-	10450 2650 10450 2750
-Wire Bus Line
-	10450 2750 10450 2850
-Wire Bus Line
-	10450 2850 10450 2950
-Wire Bus Line
-	4650 1450 4800 1450
-Wire Bus Line
-	4800 1450 4950 1450
-Wire Bus Line
-	4950 1450 5100 1450
-Wire Bus Line
-	5100 1450 5250 1450
-Wire Bus Line
-	5250 1450 5400 1450
-Wire Bus Line
-	5400 1450 5550 1450
-Wire Bus Line
-	5550 1450 5700 1450
-Wire Bus Line
-	5700 1450 10450 1450
+	4650 1450 10450 1450
 Wire Wire Line
 	4550 2350 4550 1550
@@
 	9000 4050 8750 4050
 Wire Wire Line
-	7550 4150 7500 4150
-Wire Wire Line
-	7500 4150 7450 4150
+	7450 4150 7550 4150
 Wire Wire Line
 	4450 5600 4750 5600
@@
 	4800 7150 4600 7150
 Wire Wire Line
-	2100 1300 2250 1300
-Wire Wire Line
-	2250 1300 2350 1300
+	2100 1300 2350 1300
 Wire Wire Line
 	2250 1350 2250 1300
 Connection ~ 2250 1300
 Wire Wire Line
-	1050 1650 1700 1650
-Wire Wire Line
-	1700 1650 2250 1650
-Wire Wire Line
-	1700 1600 1700 1650
-Wire Wire Line
-	1700 1650 1700 1800
-Wire Wire Line
-	800  1300 1050 1300
-Wire Wire Line
-	1050 1300 1300 1300
+	1050 1650 2250 1650
+Wire Wire Line
+	1700 1600 1700 1800
+Wire Wire Line
+	800  1300 1300 1300
 Wire Wire Line
 	1050 1350 1050 1300
@@
 	4200 6950 4150 6950
 Wire Wire Line
-	4200 6850 4200 6900
-Wire Wire Line
-	4200 6900 4200 6950
+	4200 6850 4200 6950
 Wire Wire Line
 	4200 6850 4150 6850
@@
 	7750 3550 9000 3550
 Wire Wire Line
-	4450 4650 5900 4650
-Wire Wire Line
-	5900 4650 5900 4250
-Wire Wire Line
-	5900 4250 6350 4250
-Wire Wire Line
-	4450 4750 6000 4750
-Wire Wire Line
-	6000 4750 6000 4150
-Wire Wire Line
-	6000 4150 6350 4150
+	4500 4550 4450 4550
 $EndSCHEMATC
